File: kicad/p1-interface.kicad_sch (KiCad schematic)
At the start: 6 parts, among them J1 P1 Connector, J2 Conn_01x06, J3 Conn_01x02, Q1 BC847

Commit message: Updated images and readme for rev B
Parts:
- Q1: footprint Package_TO_SOT_SMD:TSOT-23_HandSoldering -> Package_TO_SOT_SMD:SOT-23; symbol Transistor_BJT:BC547 -> Transistor_BJT:BC847
Connections:
- net GND: now also Q1.2 (E); no longer Q1.3 (E)
- net rx: now also Q1.3 (C); no longer Q1.1 (C)
- net at J1.5, R1.1: now also Q1.1 (B); no longer Q1.2 (B)
Other:
- note added: "B"
- note removed: "A"
Changed lines of the file:
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@@
     (effects (font (size 1.27 1.27)) (justify left bottom))
   )
-  (text "A" (at 269.24 194.31 0)
+  (text "B" (at 269.24 194.31 0)
     (effects (font (size 1.27 1.27)) (justify left bottom))
   )
@@
     (pin "1")
   )
-  (symbol (lib_id "Transistor_BJT:BC547") (at 158.75 101.6 0) (unit 1)
+  (symbol (lib_id "Transistor_BJT:BC847") (at 158.75 101.6 0) (unit 1)
     (in_bom yes) (on_board yes) (fields_autoplaced)
     (property "Reference" "Q1" (id 0) (at 163.6014 100.7653 0)
@@
       (effects (font (size 1.27 1.27)) (justify left))
     )
-    (property "Footprint" "Package_TO_SOT_SMD:TSOT-23_HandSoldering" (id 2) (at 163.83 103.505 0)
+    (property "Footprint" "Package_TO_SOT_SMD:SOT-23" (id 2) (at 163.83 103.505 0)
       (effects (font (size 1.27 1.27) italic) (justify left) hide)
     )
-    (property "Datasheet" "https://www.onsemi.com/pub/Collateral/BC550-D.pdf" (id 3) (at 158.75 101.6 0)
+    (property "Datasheet" "http://www.infineon.com/dgdl/Infineon-BC847SERIES_BC848SERIES_BC849SERIES_BC850SERIES-DS-v01_01-en.pdf?fileId=db3a304314dca389011541d4630a1657" (id 3) (at 158.75 101.6 0)
       (effects (font (size 1.27 1.27)) (justify left) hide)
     )
@@
     )
     (path "/2de38d86-7c82-418c-99ca-14d4f0d099d3"
-      (reference "Q1") (unit 1) (value "BC847") (footprint "Package_TO_SOT_SMD:TSOT-23_HandSoldering")
+      (reference "Q1") (unit 1) (value "BC847") (footprint "Package_TO_SOT_SMD:SOT-23")
     )
     (path "/110e359e-5f88-4430-8754-51124b3f8591"
